Commit message: Update README and configuration files to reflect joint velocity limits and goal time adjustments

File: tb20e_control/urdf/tb20e.urdf.xacro (robot description, xacro)
@@ -13,4 +13,5 @@
   <xacro:property name="bucket_position_min_deg" value="-31.0"/>
   <xacro:property name="bucket_position_max_deg" value="159.0"/>
+  <xacro:property name="joint_velocity_limit_deg_s" value="100.0"/>
   <xacro:arg name="swing_state_topic" default="/current_swing_angle"/>
   <xacro:arg name="swing_command_topic" default="/manipulated_swing_lever"/>
@@ -63,5 +64,5 @@
     <origin xyz="0 0 0.40"/>
     <axis xyz="0 0 1"/>
-    <limit effort="100.0" velocity="1.5"/>
+    <limit effort="100.0" velocity="${radians(joint_velocity_limit_deg_s)}"/>
     <dynamics damping="0.05" friction="0.02"/>
   </joint>
@@ -85,5 +86,5 @@
       upper="${radians(boom_position_max_deg)}"
       effort="100.0"
-      velocity="1.2"/>
+      velocity="${radians(joint_velocity_limit_deg_s)}"/>
     <dynamics damping="0.05" friction="0.02"/>
   </joint>
@@ -107,5 +108,5 @@
       upper="${radians(arm_position_max_deg)}"
       effort="100.0"
-      velocity="1.2"/>
+      velocity="${radians(joint_velocity_limit_deg_s)}"/>
     <dynamics damping="0.05" friction="0.02"/>
   </joint>
@@ -129,5 +130,5 @@
       upper="${radians(bucket_position_max_deg)}"
       effort="100.0"
-      velocity="1.5"/>
+      velocity="${radians(joint_velocity_limit_deg_s)}"/>
     <dynamics damping="0.05" friction="0.02"/>
   </joint>
